File: PCB Diagrams/Electronics-Power-Consumption-Meter.kicad_pcb (KiCad board)
At the start: 2 copper layers, 34 parts, among them J1 Jack_DC, J10 01x02, J11 01x02, J12 01x02, J2 01x02, J3 USB_A, J4 Jack_DC, J5 Jack_DC, J6 USB_B_Mini, J7 USB_B_Micro, J8 01x04, J9 01x02, SW1 SW_SPDT, SW2 SW_Push, U1 INA219_Module, U2 CA56-12CGKWA

Commit message: update schematics+pcb, add firmware code
Parts:
- added J3: 01x02, Connector_PinHeader_2.54mm:PinHeader_1x02_P2.54mm_Vertical, F.Cu at (161.3, 124.5)
- moved SW2 11.8 mm to (106.8, 117.9), turned to 90 degrees
- moved SW1 10.7 mm to (170.2, 130.3), turned to 90 degrees
- moved H4 5.08 mm to (100.3, 92.7)
- moved J2 4.02 mm to (179.1, 124.5), turned to 0 degrees
- moved J1 1.20 mm to (185.4, 129.2)
- moved J8 0.51 mm to (180.7, 143.0)
- moved J7 0.30 mm to (161.1, 137.9)
- moved BAT1 0.09 mm to (175.3, 118.1)
- renumbered J9 to J10, J10 to J11, J11 to J12, J12 to J13, J3 to J4, J4 to J5, J5 to J6, J6 to J7, J7 to J8, J8 to J9
Connections:
- A1 pad 25: DIG1 -> unconnected-(A1-A6-Pad25)
- A1 pad 26: SEG_A -> unconnected-(A1-A7-Pad26)
- SW1 pad 2: PWR -> Net-(J3-Pin_2)
- SW2 pad 2: 5V -> GND
Routing:
- net 5V: track 63.7 -> 12.9 mm, vias 2 -> 0
- net SEG_A: track 42.6 -> 8.67 mm
- net GND: track 392.0 -> 424.3 mm
- net DIG1: track 77.7 -> 59.8 mm
- net Net-(BAT1-+): track 23.6 -> 9.19 mm
- net Net-(SW1-A): track 29.9 -> 16.1 mm
- net Net-(J3-Pin_2): track 0.00 -> 9.42 mm
- net PWR: track 39.6 -> 35.9 mm
- net Net-(A1-A0): track 26.4 -> 29.6 mm
- net VIN+: track 107.1 -> 104.4 mm
- net VIN-: track 200.9 -> 203.3 mm
- net I2C_SDA: track 21.8 -> 23.0 mm
- net I2C_SCL: track 18.3 -> 19.6 mm
- net DATA1-: track 102.0 -> 103.0 mm
- net DATA1+: track 101.8 -> 102.8 mm
Other:
- board outline added: 99.1 x 109.2 mm

Commit message: update firmware
Parts:
- added R10: R470, Resistor_THT:R_Axial_DIN0207_L6.3mm_D2.5mm_P2.54mm_Vertical, F.Cu at (124.5, 115.6)
- added R11: R470, Resistor_THT:R_Axial_DIN0207_L6.3mm_D2.5mm_P2.54mm_Vertical, F.Cu at (128.3, 115.6)
- R1, R2, R3, R4, R5, R6, R7, R8: footprint Resistor_THT:R_Axial_DIN0207_L6.3mm_D2.5mm_P7.62mm_Horizontal -> Resistor_THT:R_Axial_DIN0207_L6.3mm_D2.5mm_P2.54mm_Vertical
- R9: value R1K -> R470; footprint Resistor_THT:R_Axial_DIN0207_L6.3mm_D2.5mm_P7.62mm_Horizontal -> Resistor_THT:R_Axial_DIN0207_L6.3mm_D2.5mm_P2.54mm_Vertical
- moved D3 25.4 mm to (146.1, 124.5)
- moved D2 17.6 mm to (141.0, 124.5)
- moved U1 10.9 mm to (138.4, 108.0), turned to 180 degrees
- moved D1 10.5 mm to (135.9, 124.5)
- moved SW2 8.13 mm to (113.1, 112.8)
- moved R9 6.84 mm to (120.7, 115.6), turned to -90 degrees
- moved A1 5.08 mm to (148.6, 78.7)
- moved R1 4.70 mm to (110.5, 71.5)
- moved R2 4.70 mm to (114.3, 71.5)
- moved R3 4.70 mm to (118.1, 71.5)
- moved R4 4.70 mm to (121.9, 71.5)
- moved R5 4.70 mm to (125.7, 71.5)
- moved R6 4.70 mm to (129.5, 71.5)
- moved R7 4.70 mm to (133.3, 71.5)
- moved R8 4.70 mm to (143.5, 71.5)
- renumbered D3 to D1, D1 to D3
Connections:
- D2 pad 1: Net-(D1-K) -> Net-(D2-K)
- D3 pad 1: Net-(D1-K) -> Net-(D3-K)
Routing:
- net GND: track 424.3 -> 383.1 mm
- net Net-(D1-K): track 27.0 -> 0.00 mm
- net Net-(A1-A1): track 24.2 -> 2.54 mm
- net Net-(A1-A0): track 29.6 -> 11.7 mm
- net Net-(A1-A2): track 16.1 -> 2.54 mm
- net I2C_SDA: track 23.0 -> 10.5 mm
- net Net-(A1-A3): track 9.42 -> 0.00 mm
- net I2C_SCL: track 19.6 -> 10.5 mm
- net VIN-: track 203.3 -> 197.1 mm
- net DIG3: track 43.5 -> 38.4 mm
- net DIG2: track 43.5 -> 38.4 mm
- net DIG1: track 59.8 -> 54.7 mm
- net DIG4: track 25.5 -> 20.4 mm
- net VIN+: track 104.4 -> 99.9 mm
- net 5V: track 12.9 -> 8.67 mm
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
Commit message: update schematics and PCB
Parts:
- U2: value CA56-12CGKWA -> Display_5641BS
- moved D1 34.2 mm to (110.5, 101.6)
- moved D2 32.3 mm to (118.1, 101.6)
- moved D3 30.6 mm to (125.7, 101.6)
- moved R9 14.4 mm to (110.5, 105.4)
- moved R10 12.0 mm to (118.1, 105.4)
- moved R11 10.5 mm to (125.7, 105.4)
- moved U1 6.48 mm to (144.8, 109.2), turned to -90 degrees
- moved SW2 2.97 mm to (115.7, 114.3), turned to 0 degrees
- moved J3 2.84 mm to (158.8, 125.7), turned to 90 degrees
- moved J2 1.27 mm to (179.1, 125.7), turned to -90 degrees
Connections:
- D1 pad 2: Net-(A1-A1) -> Net-(A1-A0)
- D2 pad 2: Net-(A1-A2) -> Net-(A1-A1)
- D3 pad 2: Net-(A1-A3) -> Net-(A1-A2)
- SW2 pad 1: Net-(A1-A0) -> Net-(A1-A3)
Routing:
- net GND: track 383.1 -> 498.4 mm, vias 3 -> 5
- net Net-(A1-A3): track 0.00 -> 34.0 mm
- net VIN+: track 99.9 -> 115.7 mm
- net I2C_SDA: track 10.5 -> 20.6 mm
- net VIN-: track 197.1 -> 205.2 mm
- net I2C_SCL: track 10.5 -> 16.3 mm
- net Net-(A1-A1): track 2.54 -> 7.93 mm
- net DATA1-: track 103.0 -> 98.8 mm
- net DATA1+: track 102.8 -> 98.7 mm
- net Net-(D3-K): track 0.00 -> 3.81 mm
- net Net-(D2-K): track 0.00 -> 3.81 mm
- net Net-(D1-K): track 0.00 -> 3.81 mm
- net Net-(BAT1-+): track 9.19 -> 6.57 mm
- net Net-(A1-A2): track 2.54 -> 5.08 mm
- net 5V: track 8.67 -> 10.5 mm
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
Commit message: update schematics and PCB
Parts:
- removed H4: MountingHole, MountingHole:MountingHole_2mm
- moved R3 3.87 mm to (115.6, 68.6)
- moved R4 3.87 mm to (119.4, 68.6)
- moved R5 3.87 mm to (123.2, 68.6)
- moved R1 3.87 mm to (108.0, 68.6)
- moved R2 3.87 mm to (111.8, 68.6)
- moved R6 3.87 mm to (127.0, 68.6)
- moved R7 3.87 mm to (130.8, 68.6)
- moved R8 3.18 mm to (142.2, 68.6)
- moved H1 2.54 mm to (100.3, 36.8)
- moved H2 2.54 mm to (191.8, 36.8)
- moved J6 2.10 mm to (144.3, 135.7)
- moved J5 2.10 mm to (127.8, 135.7)
- moved J8 1.53 mm to (180.7, 144.5)
- moved J7 1.29 mm to (161.1, 139.2)
- moved J4 1.27 mm to (104.6, 135.6)
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Routing:
- net GND: track 498.4 -> 481.2 mm
- net VIN+: track 115.7 -> 127.0 mm
- net VIN-: track 205.2 -> 213.3 mm
- net DATA1-: track 98.8 -> 103.9 mm
- net SEG_B: track 7.51 -> 11.7 mm
- net SEG_A: track 8.04 -> 12.3 mm
- net SEG_E: track 7.24 -> 11.2 mm
- net DATA1+: track 98.7 -> 102.4 mm
- net DIG1: track 54.7 -> 57.7 mm
- net SEG_D: track 7.77 -> 10.7 mm
- net Net-(U2-g): track 7.78 -> 5.08 mm
- net SEG_F: track 9.09 -> 11.7 mm
- net Net-(U2-b): track 26.2 -> 24.0 mm
- net SEG_G: track 9.09 -> 11.2 mm
- net SEG_C: track 8.56 -> 10.7 mm
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Other:
- board size 99.1 x 109.2 mm -> 99.1 x 113 mm
