File: PCB Diagrams/Electronics-Power-Consumption-Meter.kicad_sch (KiCad schematic)
At the start: 0 parts

Commit message: adding schematics and PCB
Parts:
- added A1: Arduino_Nano_v3.x, Custom:Arduino_Nano_v3, symbol MCU_Module:Arduino_Nano_v3.x
- added BAT1: BAT_18650, Custom:BatteryHolder_18650_X2, symbol Device:Battery
- added D1, D2, D3: LED, LED_THT:LED_D3.0mm, symbol PCM_SparkFun-LED:LED
- added H1, H2, H3, H4: MountingHole, MountingHole:MountingHole_2mm, symbol Mechanical:MountingHole
- added J1, J4, J5: Jack_DC, Connector_BarrelJack:BarrelJack_Horizontal, symbol Connector:Barrel_Jack_MountingPin
- added J10, J11, J12, J9: 01x02, Connector_PinSocket_2.54mm:PinSocket_1x02_P2.54mm_Vertical, symbol Connector_Generic:Conn_01x02
- added J2: 01x02, Connector_PinHeader_2.54mm:PinHeader_1x02_P2.54mm_Vertical, symbol Connector:Conn_01x02_Pin
- added J3: USB_A, Connector_USB:USB_A_Molex_67643_Horizontal, symbol Connector:USB_A
- added J6: USB_B_Mini, Custom:USB_B_Mini_OTG_THT_Molex_548190519, symbol Connector:USB_B_Mini
- added J7: USB_B_Micro, Custom:USB_B_Micro_THT_Amphenol_101181940011LF, symbol Connector:USB_B_Micro
- added J8: 01x04, Connector_PinSocket_2.54mm:PinSocket_1x04_P2.54mm_Vertical, symbol Connector_Generic:Conn_01x04
- added R1, R2, R3, R4, R5, R6, R7, R8: R470, Resistor_THT:R_Axial_DIN0207_L6.3mm_D2.5mm_P7.62mm_Horizontal, symbol Device:R
- added R9: R1K, Resistor_THT:R_Axial_DIN0207_L6.3mm_D2.5mm_P7.62mm_Horizontal, symbol Device:R
- added SW1: SW_SPDT, Button_Switch_THT:SW_Slide_SPDT_Straight_CK_OS102011MS2Q, symbol Switch:SW_SPDT
- added SW2: SW_Push, Button_Switch_THT:SW_PUSH-12mm_Wuerth-430476085716, symbol Switch:SW_Push
- added U1: INA219_Module, Custom:INA219_Module_Adafruit, symbol Custom:INA219_Module
- added U2: CA56-12CGKWA, Display_7Segment:CA56-12CGKWA, symbol Display_Character:CA56-12CGKWA
Connections:
- new net: R8.2, U2.7 (b)
- new net: R5.2, U2.3 (DPX)
- new net: R2.2, U2.10 (f)
- new net: A1.19 (A0), SW2.1
- new net: A1.20 (A1), D3.2 (A)
- new net: A1.21 (A2), D2.2 (A)
- new net: A1.22 (A3), D1.2 (A)
- new net: R3.2, U2.1 (e)
- new net: R1.2, U2.11 (a)
- new net: R4.2, U2.2 (d)
- new net: R6.2, U2.4 (c)
- new net: R7.2, U2.5 (g)
- new net: J1.1, SW1.1 (A)
- new net: BAT1.1 (+), J2.2 (Pin_2), SW1.3 (C)
- new net: D1.1 (K), D2.1 (K), D3.1 (K), R9.1
- new net 5V: A1.27 (+5V), SW2.2, U1.1 (VCC)
- new net DATA1+: J3.3 (D+), J8.2 (Pin_2)
- new net DATA1-: J3.2 (D-), J8.3 (Pin_3)
- new net DIG1: A1.25 (A6), U2.12 (CA1)
- new net DIG2: A1.7 (D4), U2.9 (CA2)
- new net DIG3: A1.6 (D3), U2.8 (CA3)
- new net DIG4: A1.8 (D5), U2.6 (CA4)
- new net GND: A1.29 (GND), A1.4 (GND), BAT1.2 (-), J1.2, J10.1 (Pin_1), J11.1 (Pin_1), J12.1 (Pin_1), J2.1 (Pin_1), J3.4 (GND), J4.2, J5.2, J6.5 (GND), J7.5 (GND), J8.1 (Pin_1), J9.1 (Pin_1), R9.2, U1.2 (GND)
- new net I2C_SCL: A1.24 (A5), U1.3 (SCL)
- new net I2C_SDA: A1.23 (A4), U1.4 (SDA)
- new net PWR: A1.30 (VIN), SW1.2 (B)
- new net SEG_A: A1.26 (A7), R1.1
- new net SEG_B: A1.14 (D11), R2.1
- new net SEG_C: A1.10 (D7), R6.1
- new net SEG_D: A1.12 (D9), R4.1
- new net SEG_E: A1.13 (D10), R3.1
- new net SEG_F: A1.5 (D2), R8.1
- new net SEG_G: A1.9 (D6), R7.1
- new net SEG_P: A1.11 (D8), R5.1
- new net VIN+: J3.1 (VBUS), J4.1, J5.1, J6.1 (VBUS), J7.1 (VBUS), U1.6 (VIN+)
- new net VIN-: J10.2 (Pin_2), J11.2 (Pin_2), J12.2 (Pin_2), J8.4 (Pin_4), J9.2 (Pin_2), U1.5 (VIN-)

Commit message: update schematics+pcb, add firmware code
Parts:
- added J3: 01x02, Connector_PinHeader_2.54mm:PinHeader_1x02_P2.54mm_Vertical, symbol Connector:Conn_01x02_Pin
- renumbered J9 to J10, J10 to J11, J11 to J12, J12 to J13, J3 to J4, J4 to J5, J5 to J6, J6 to J7, J7 to J8, J8 to J9
Connections:
- net 5V: no longer SW2.2
- net DIG1: now also A1.16 (D13); no longer A1.25 (A6)
- net GND: now also SW2.2
- net PWR: now also J3.1 (Pin_1); no longer SW1.2 (B)
- net SEG_A: now also A1.15 (D12); no longer A1.26 (A7)
- new net: J3.2 (Pin_2), SW1.2 (B)
Changed lines of the file:
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@@
 	(wire
 		(pts
-			(xy 60.96 88.9) (xy 64.77 88.9)
-		)
-		(stroke
-			(width 0)
-			(type default)
-		)
-	)
-	(wire
-		(pts
 			(xy 143.51 113.03) (xy 143.51 124.46)
 		)
@@
 	(wire
 		(pts
-			(xy 128.27 50.8) (xy 125.73 50.8)
+			(xy 125.73 58.42) (xy 128.27 58.42)
 		)
 		(stroke
@@
 	(wire
 		(pts
-			(xy 125.73 58.42) (xy 128.27 58.42)
+			(xy 153.67 58.42) (xy 156.21 58.42)
 		)
 		(stroke
@@
 	(wire
 		(pts
-			(xy 153.67 58.42) (xy 156.21 58.42)
+			(xy 64.77 83.82) (xy 64.77 86.36)
 		)
 		(stroke
@@
 	(wire
 		(pts
-			(xy 64.77 83.82) (xy 64.77 86.36)
+			(xy 106.68 113.03) (xy 106.68 128.27)
 		)
 		(stroke
@@
 	(wire
 		(pts
-			(xy 106.68 113.03) (xy 106.68 128.27)
+			(xy 135.89 148.59) (xy 149.86 148.59)
 		)
 		(stroke
@@
 	(wire
 		(pts
-			(xy 135.89 148.59) (xy 149.86 148.59)
+			(xy 153.67 50.8) (xy 156.21 50.8)
 		)
 		(stroke
@@
 	(wire
 		(pts
-			(xy 50.8 69.85) (xy 50.8 81.28)
+			(xy 63.5 92.71) (xy 63.5 88.9)
+		)
+		(stroke
+			(width 0)
+			(type default)
+		)
+	)
+	(wire
+		(pts
+			(xy 50.8 69.85) (xy 50.8 78.74)
 		)
 		(stroke
@@
 	(wire
 		(pts
-			(xy 128.27 53.34) (xy 125.73 53.34)
+			(xy 63.5 88.9) (xy 64.77 88.9)
 		)
 		(stroke
@@
 	(wire
 		(pts
+			(xy 153.67 53.34) (xy 156.21 53.34)
+		)
+		(stroke
+			(width 0)
+			(type default)
+		)
+	)
+	(wire
+		(pts
 			(xy 123.19 113.03) (xy 143.51 113.03)
 		)
@@
 		)
 	)
-	(global_label "SEG_A"
+	(global_label "GND"
 		(shape input)
-		(at 125.73 50.8 180)
+		(at 111.76 68.58 180)
 		(fields_autoplaced yes)
 		(effects
@@
 		)
 		(property "Intersheetrefs" "${INTERSHEET_REFS}"
-			(at 117.0601 50.8 0)
+			(at 104.9043 68.58 0)
 			(effects
 				(font
@@
 		)
 	)
+	(global_label "DIG1"
+		(shape input)
+		(at 156.21 50.8 0)
+		(fields_autoplaced yes)
+		(effects
+			(font
+				(size 1.27 1.27)
+			)
+			(justify left)
+		)
+		(property "Intersheetrefs" "${INTERSHEET_REFS}"
+			(at 163.5495 50.8 0)
+			(effects
+				(font
+					(size 1.27 1.27)
+				)
+				(justify left)
+				(hide yes)
+			)
+		)
+	)
 	(global_label "GND"
 		(shape input)
@@
 		)
 	)
+	(global_label "SEG_A"
+		(shape input)
+		(at 156.21 53.34 0)
+		(fields_autoplaced yes)
+		(effects
+			(font
+				(size 1.27 1.27)
+			)
+			(justify left)
+		)
+		(property "Intersheetrefs" "${INTERSHEET_REFS}"
+			(at 164.8799 53.34 0)
+			(effects
+				(font
+					(size 1.27 1.27)
+				)
+				(justify left)
+				(hide yes)
+			)
+		)
+	)
 	(global_label "I2C_SCL"
 		(shape input)
@@
 		)
 	)
-	(global_label "5V"
-		(shape input)
-		(at 111.76 68.58 180)
-		(fields_autoplaced yes)
-		(effects
-			(font
-				(size 1.27 1.27)
-			)
-			(justify right)
-		)
-		(property "Intersheetrefs" "${INTERSHEET_REFS}"
-			(at 106.4767 68.58 0)
-			(effects
-				(font
-					(size 1.27 1.27)
-				)
-				(justify right)
-				(hide yes)
-			)
-		)
-	)
 	(global_label "GND"
 		(shape input)
@@
 		)
 	)
-	(global_label "DIG1"
-		(shape input)
-		(at 125.73 53.34 180)
-		(fields_autoplaced yes)
-		(effects
-			(font
-				(size 1.27 1.27)
-			)
-			(justify right)
-		)
-		(property "Intersheetrefs" "${INTERSHEET_REFS}"
-			(at 118.3905 53.34 0)
-			(effects
-				(font
-					(size 1.27 1.27)
-				)
-				(justify right)
-				(hide yes)
-			)
-		)
-	)
 	(global_label "GND"
 		(shape input)
@@
 	(global_label "GND"
 		(shape input)
-		(at 60.96 88.9 180)
+		(at 63.5 92.71 270)
 		(fields_autoplaced yes)
 		(effects
@@
 		)
 		(property "Intersheetrefs" "${INTERSHEET_REFS}"
-			(at 54.1043 88.9 0)
+			(at 63.5 99.5657 90)
 			(effects
 				(font
@@
 		(dnp no)
 		(fields_autoplaced yes)
-		(property "Reference" "J6"
+		(property "Reference" "J7"
 			(at 115.57 116.84 0)
 			(effects
@@
 			(project ""
 				(path "/04a21a1e-c762-45c9-8522-5107851ca11f"
-					(reference "J6")
+					(reference "J7")
 					(unit 1)
 				)
@@
 	)
 	(symbol
+		(lib_id "Connector:Conn_01x02_Pin")
+		(at 45.72 78.74 0)
+		(unit 1)
+		(exclude_from_sim no)
+		(in_bom yes)
+		(on_board yes)
+		(dnp no)
+		(property "Reference" "J3"
+			(at 46.99 83.058 0)
+			(effects
+				(font
+					(size 1.27 1.27)
+				)
+			)
+		)
+		(property "Value" "01x02"
+			(at 46.99 85.09 0)
+			(effects
+				(font
+					(size 1.27 1.27)
+				)
+			)
+		)
+		(property "Footprint" "Connector_PinHeader_2.54mm:PinHeader_1x02_P2.54mm_Vertical"
+			(at 45.72 78.74 0)
+			(effects
+				(font
+					(size 1.27 1.27)
+				)
+				(hide yes)
+			)
+		)
+		(property "Datasheet" "~"
+			(at 45.72 78.74 0)
+			(effects
+				(font
+					(size 1.27 1.27)
+				)
+				(hide yes)
+			)
+		)
+		(property "Description" "Generic connector, single row, 01x02, script generated"
+			(at 45.72 78.74 0)
+			(effects
+				(font
+					(size 1.27 1.27)
+				)
+				(hide yes)
+			)
+		)
+		(pin "2"
+		)
+		(pin "1"
+		)
+		(instances
+			(project "Electronics-Power-Consumption-Meter"
+				(path "/04a21a1e-c762-45c9-8522-5107851ca11f"
+					(reference "J3")
+					(unit 1)
+				)
+			)
+		)
+	)
+	(symbol
 		(lib_id "MCU_Module:Arduino_Nano_v3.x")
 		(at 140.97 68.58 180)
@@
 		(on_board yes)
 		(dnp no)
-		(property "Reference" "J4"
+		(property "Reference" "J5"
 			(at 82.55 121.92 0)
 			(effects
@@
 			(project ""
 				(path "/04a21a1e-c762-45c9-8522-5107851ca11f"
-					(reference "J4")
+					(reference "J5")
 					(unit 1)
 				)
@@
 		(on_board yes)
 		(dnp no)
-		(property "Reference" "J5"
+		(property "Reference" "J6"
 			(at 99.06 121.92 0)
 			(effects
@@
 			(project "Electronics-Power-Consumption-Meter"
 				(path "/04a21a1e-c762-45c9-8522-5107851ca11f"
-					(reference "J5")
+					(reference "J6")
 					(unit 1)
 				)
@@
 		(on_board yes)
 		(dnp no)
-		(property "Reference" "J11"
+		(property "Reference" "J12"
 			(at 205.232 126.492 0)
 			(effects
@@
 			(project "Electronics-Power-Consumption-Meter"
 				(path "/04a21a1e-c762-45c9-8522-5107851ca11f"
-					(reference "J11")
+					(reference "J12")
 					(unit 1)
 				)
@@
 		(dnp no)
 		(fields_autoplaced yes)
-		(property "Reference" "J3"
+		(property "Reference" "J4"
 			(at 62.23 116.84 0)
 			(effects
@@
 			(project ""
 				(path "/04a21a1e-c762-45c9-8522-5107851ca11f"
-					(reference "J3")
+					(reference "J4")
 					(unit 1)
 				)
@@
 		(dnp no)
 		(fields_autoplaced yes)
-		(property "Reference" "J7"
+		(property "Reference" "J8"
 			(at 135.89 116.84 0)
 			(effects
@@
 			(project ""
 				(path "/04a21a1e-c762-45c9-8522-5107851ca11f"
-					(reference "J7")
+					(reference "J8")
 					(unit 1)
 				)
@@
 		(on_board yes)
 		(dnp no)
-		(property "Reference" "J12"
+		(property "Reference" "J13"
 			(at 219.202 126.492 0)
 			(effects
@@
 			(project "Electronics-Power-Consumption-Meter"
 				(path "/04a21a1e-c762-45c9-8522-5107851ca11f"
-					(reference "J12")
+					(reference "J13")
 					(unit 1)
 				)
@@
 		(dnp no)
 		(property "Reference" "J2"
-			(at 67.056 90.932 0)
+			(at 67.818 90.424 0)
 			(effects
 				(font
@@
 		)
 		(property "Value" "01x02"
-			(at 67.31 92.964 0)
+			(at 67.818 92.456 0)
 			(effects
 				(font
@@
 		(on_board yes)
 		(dnp no)
-		(property "Reference" "J9"
+		(property "Reference" "J10"
 			(at 184.912 126.492 0)
 			(effects
@@
 			(project ""
 				(path "/04a21a1e-c762-45c9-8522-5107851ca11f"
-					(reference "J9")
+					(reference "J10")
 					(unit 1)
 				)
@@
 		(on_board yes)
 		(dnp no)
-		(property "Reference" "J10"
+		(property "Reference" "J11"
 			(at 195.072 126.492 0)
 			(effects
@@
 			(project "Electronics-Power-Consumption-Meter"
 				(path "/04a21a1e-c762-45c9-8522-5107851ca11f"
-					(reference "J10")
+					(reference "J11")
 					(unit 1)
 				)
@@
 		(on_board yes)
 		(dnp no)
-		(property "Reference" "J8"
+		(property "Reference" "J9"
 			(at 170.18 123.952 0)
 			(effects
@@
 			(project "Electronics-Power-Consumption-Meter"
 				(path "/04a21a1e-c762-45c9-8522-5107851ca11f"
-					(reference "J8")
+					(reference "J9")
 					(unit 1)
 				)

Commit message: update firmware
Parts:
- added R10, R11: R470, Resistor_THT:R_Axial_DIN0207_L6.3mm_D2.5mm_P2.54mm_Vertical, symbol Device:R
- R1, R2, R3, R4, R5, R6, R7, R8: footprint Resistor_THT:R_Axial_DIN0207_L6.3mm_D2.5mm_P7.62mm_Horizontal -> Resistor_THT:R_Axial_DIN0207_L6.3mm_D2.5mm_P2.54mm_Vertical
- R9: value R1K -> R470; footprint Resistor_THT:R_Axial_DIN0207_L6.3mm_D2.5mm_P7.62mm_Horizontal -> Resistor_THT:R_Axial_DIN0207_L6.3mm_D2.5mm_P2.54mm_Vertical
- renumbered D3 to D1, D1 to D3
Connections:
- net GND: now also R10.2, R11.2
- net at D1.1 (K), R9.1: no longer D2.1 (K), D3.1 (K)
- new net: D2.1 (K), R10.1
- new net: D3.1 (K), R11.1
Other:
- moved on the sheet: R9
Changed lines of the file:
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@@
 	)
 	(junction
-		(at 101.6 53.34)
-		(diameter 0)
-		(color 0 0 0 0)
-	)
-	(junction
-		(at 105.41 53.34)
+		(at 105.41 43.18)
 		(diameter 0)
 		(color 0 0 0 0)
@@
 	(wire
 		(pts
-			(xy 109.22 53.34) (xy 105.41 53.34)
+			(xy 198.12 113.03) (xy 208.28 113.03)
 		)
 		(stroke
@@
 	(wire
 		(pts
-			(xy 198.12 113.03) (xy 208.28 113.03)
+			(xy 101.6 43.18) (xy 105.41 43.18)
 		)
 		(stroke
@@
 	(wire
 		(pts
+			(xy 105.41 40.64) (xy 105.41 43.18)
+		)
+		(stroke
+			(width 0)
+			(type default)
+		)
+	)
+	(wire
+		(pts
 			(xy 175.26 63.5) (xy 177.8 63.5)
 		)
@@
 	(wire
 		(pts
-			(xy 101.6 40.64) (xy 101.6 43.18)
+			(xy 101.6 43.18) (xy 101.6 45.72)
 		)
 		(stroke
@@
 	(wire
 		(pts
-			(xy 105.41 53.34) (xy 101.6 53.34)
-		)
-		(stroke
-			(width 0)
-			(type default)
-		)
-	)
-	(wire
-		(pts
 			(xy 222.25 132.08) (xy 222.25 148.59)
 		)
@@
 	(wire
 		(pts
+			(xy 109.22 43.18) (xy 109.22 45.72)
+		)
+		(stroke
+			(width 0)
+			(type default)
+		)
+	)
+	(wire
+		(pts
 			(xy 175.26 55.88) (xy 177.8 55.88)
 		)
@@
 	(wire
 		(pts
-			(xy 50.8 69.85) (xy 50.8 78.74)
+			(xy 105.41 43.18) (xy 109.22 43.18)
 		)
 		(stroke
@@
 	(wire
 		(pts
-			(xy 198.12 113.03) (xy 198.12 129.54)
+			(xy 50.8 69.85) (xy 50.8 78.74)
 		)
 		(stroke
@@
 	(wire
 		(pts
-			(xy 222.25 148.59) (xy 227.33 148.59)
+			(xy 198.12 113.03) (xy 198.12 129.54)
 		)
 		(stroke
@@
 	(wire
 		(pts
-			(xy 175.26 68.58) (xy 177.8 68.58)
+			(xy 222.25 148.59) (xy 227.33 148.59)
 		)
 		(stroke
@@
 	(wire
 		(pts
-			(xy 198.12 132.08) (xy 198.12 148.59)
+			(xy 175.26 68.58) (xy 177.8 68.58)
 		)
 		(stroke
@@
 	(wire
 		(pts
-			(xy 106.68 113.03) (xy 123.19 113.03)
+			(xy 198.12 132.08) (xy 198.12 148.59)
 		)
 		(stroke
@@
 	(wire
 		(pts
-			(xy 153.67 66.04) (xy 156.21 66.04)
+			(xy 106.68 113.03) (xy 123.19 113.03)
 		)
 		(stroke
@@
 	(wire
 		(pts
-			(xy 101.6 50.8) (xy 101.6 53.34)
+			(xy 153.67 66.04) (xy 156.21 66.04)
 		)
 		(stroke
@@
 	(wire
 		(pts
+			(xy 105.41 43.18) (xy 105.41 45.72)
+		)
+		(stroke
+			(width 0)
+			(type default)
+		)
+	)
+	(wire
+		(pts
 			(xy 72.39 127) (xy 72.39 129.54)
 		)
@@
 		)
 	)
+	(global_label "GND"
+		(shape input)
+		(at 105.41 40.64 90)
+		(fields_autoplaced yes)
+		(effects
+			(font
+				(size 1.27 1.27)
+			)
+			(justify left)
+		)
+		(property "Intersheetrefs" "${INTERSHEET_REFS}"
+			(at 105.41 33.7843 90)
+			(effects
+				(font
+					(size 1.27 1.27)
+				)
+				(justify left)
+				(hide yes)
+			)
+		)
+	)
 	(global_label "SEG_E"
 		(shape input)
@@
 		)
 	)
-	(global_label "GND"
-		(shape input)
-		(at 101.6 40.64 90)
-		(fields_autoplaced yes)
-		(effects
-			(font
-				(size 1.27 1.27)
-			)
-			(justify left)
-		)
-		(property "Intersheetrefs" "${INTERSHEET_REFS}"
-			(at 101.6 33.7843 90)
-			(effects
-				(font
-					(size 1.27 1.27)
-				)
-				(justify left)
-				(hide yes)
-			)
-		)
-	)
 	(global_label "SEG_C"
 		(shape input)
@@
 			)
 		)
-		(property "Footprint" "Resistor_THT:R_Axial_DIN0207_L6.3mm_D2.5mm_P7.62mm_Horizontal"
+		(property "Footprint" "Resistor_THT:R_Axial_DIN0207_L6.3mm_D2.5mm_P2.54mm_Vertical"
 			(at 181.61 60.198 90)
 			(effects
@@
 			)
 		)
-		(property "Footprint" "Resistor_THT:R_Axial_DIN0207_L6.3mm_D2.5mm_P7.62mm_Horizontal"
+		(property "Footprint" "Resistor_THT:R_Axial_DIN0207_L6.3mm_D2.5mm_P2.54mm_Vertical"
 			(at 181.61 75.438 90)
 			(effects
@@
 			)
 		)
-		(property "Footprint" "Resistor_THT:R_Axial_DIN0207_L6.3mm_D2.5mm_P7.62mm_Horizontal"
+		(property "Footprint" "Resistor_THT:R_Axial_DIN0207_L6.3mm_D2.5mm_P2.54mm_Vertical"
 			(at 181.61 70.358 90)
 			(effects
@@
 			)
 		)
-		(property "Footprint" "Resistor_THT:R_Axial_DIN0207_L6.3mm_D2.5mm_P7.62mm_Horizontal"
+		(property "Footprint" "Resistor_THT:R_Axial_DIN0207_L6.3mm_D2.5mm_P2.54mm_Vertical"
 			(at 181.61 72.898 90)
 			(effects
@@
 			)
 		)
-		(property "Footprint" "Resistor_THT:R_Axial_DIN0207_L6.3mm_D2.5mm_P7.62mm_Horizontal"
+		(property "Footprint" "Resistor_THT:R_Axial_DIN0207_L6.3mm_D2.5mm_P2.54mm_Vertical"
 			(at 181.61 62.738 90)
 			(effects
@@
 	)
 	(symbol
+		(lib_id "Device:R")
+		(at 105.41 49.53 180)
+		(unit 1)
+		(exclude_from_sim no)
+		(in_bom yes)
+		(on_board yes)
+		(dnp no)
+		(property "Reference" "R10"
+			(at 105.41 49.53 90)
+			(effects
+				(font
+					(size 1.27 1.27)
+				)
+			)
+		)
+		(property "Value" "R470"
+			(at 108.966 49.276 90)
+			(effects
+				(font
+					(size 1.27 1.27)
+				)
+				(hide yes)
+			)
+		)
+		(property "Footprint" "Resistor_THT:R_Axial_DIN0207_L6.3mm_D2.5mm_P2.54mm_Vertical"
+			(at 107.188 49.53 90)
+			(effects
+				(font
+					(size 1.27 1.27)
+				)
+				(hide yes)
+			)
+		)
+		(property "Datasheet" "~"
+			(at 105.41 49.53 0)
+			(effects
+				(font
+					(size 1.27 1.27)
+				)
+				(hide yes)
+			)
+		)
+		(property "Description" "Resistor"
+			(at 105.41 49.53 0)
+			(effects
+				(font
+					(size 1.27 1.27)
+				)
+				(hide yes)
+			)
+		)
+		(pin "1"
+		)
+		(pin "2"
+		)
+		(instances
+			(project "Electronics-Power-Consumption-Meter"
+				(path "/04a21a1e-c762-45c9-8522-5107851ca11f"
+					(reference "R10")
+					(unit 1)
+				)
+			)
+		)
+	)
+	(symbol
 		(lib_id "Connector:Barrel_Jack_MountingPin")
 		(at 99.06 130.81 0)
@@
 	(symbol
 		(lib_id "Device:R")
-		(at 101.6 46.99 180)
+		(at 101.6 49.53 180)
 		(unit 1)
 		(exclude_from_sim no)
@@
 		(dnp no)
 		(property "Reference" "R9"
-			(at 101.6 46.99 90)
+			(at 101.6 49.53 90)
 			(effects
 				(font
@@
 			)
 		)
-		(property "Value" "R1K"
-			(at 105.156 46.736 90)
+		(property "Value" "R470"
+			(at 105.156 49.276 90)
 			(effects
 				(font
@@
 			)
 		)
-		(property "Footprint" "Resistor_THT:R_Axial_DIN0207_L6.3mm_D2.5mm_P7.62mm_Horizontal"
-			(at 103.378 46.99 90)
+		(property "Footprint" "Resistor_THT:R_Axial_DIN0207_L6.3mm_D2.5mm_P2.54mm_Vertical"
+			(at 103.378 49.53 90)
 			(effects
 				(font
@@
 		)
 		(property "Datasheet" "~"
-			(at 101.6 46.99 0)
+			(at 101.6 49.53 0)
 			(effects
 				(font
@@
 		)
 		(property "Description" "Resistor"
-			(at 101.6 46.99 0)
+			(at 101.6 49.53 0)
 			(effects
 				(font
@@
 			)
 		)
-		(property "Footprint" "Resistor_THT:R_Axial_DIN0207_L6.3mm_D2.5mm_P7.62mm_Horizontal"
+		(property "Footprint" "Resistor_THT:R_Axial_DIN0207_L6.3mm_D2.5mm_P2.54mm_Vertical"
 			(at 181.61 57.658 90)
 			(effects
@@
 	)
 	(symbol
+		(lib_id "Device:R")
+		(at 109.22 49.53 180)
+		(unit 1)
+		(exclude_from_sim no)
+		(in_bom yes)
+		(on_board yes)
+		(dnp no)
+		(property "Reference" "R11"
+			(at 109.22 49.53 90)
+			(effects
+				(font
+					(size 1.27 1.27)
+				)
+			)
+		)
+		(property "Value" "R470"
+			(at 112.776 49.276 90)
+			(effects
+				(font
+					(size 1.27 1.27)
+				)
+				(hide yes)
+			)
+		)
+		(property "Footprint" "Resistor_THT:R_Axial_DIN0207_L6.3mm_D2.5mm_P2.54mm_Vertical"
+			(at 110.998 49.53 90)
+			(effects
+				(font
+					(size 1.27 1.27)
+				)
+				(hide yes)
+			)
+		)
+		(property "Datasheet" "~"
+			(at 109.22 49.53 0)
+			(effects
+				(font
+					(size 1.27 1.27)
+				)
+				(hide yes)
+			)
+		)
+		(property "Description" "Resistor"
+			(at 109.22 49.53 0)
+			(effects
+				(font
+					(size 1.27 1.27)
+				)
+				(hide yes)
+			)
+		)
+		(pin "1"
+		)
+		(pin "2"
+		)
+		(instances
+			(project "Electronics-Power-Consumption-Meter"
+				(path "/04a21a1e-c762-45c9-8522-5107851ca11f"
+					(reference "R11")
+					(unit 1)
+				)
+			)
+		)
+	)
+	(symbol
 		(lib_id "Connector_Generic:Conn_01x02")
 		(at 193.04 132.08 180)
@@
 		(on_board yes)
 		(dnp no)
-		(property "Reference" "D3"
+		(property "Reference" "D1"
 			(at 101.854 56.134 90)
 			(effects
@@
 		)
 		(instances
-			(project ""
+			(project "Electronics-Power-Consumption-Meter"
 				(path "/04a21a1e-c762-45c9-8522-5107851ca11f"
-					(reference "D3")
+					(reference "D1")
 					(unit 1)
 				)
@@
 		(on_board yes)
 		(dnp no)
-		(property "Reference" "D1"
+		(property "Reference" "D3"
 			(at 109.474 56.134 90)
 			(effects
@@
 			(project "Electronics-Power-Consumption-Meter"
 				(path "/04a21a1e-c762-45c9-8522-5107851ca11f"
-					(reference "D1")
+					(reference "D3")
 					(unit 1)
 				)
@@
 			)
 		)
-		(property "Footprint" "Resistor_THT:R_Axial_DIN0207_L6.3mm_D2.5mm_P7.62mm_Horizontal"
+		(property "Footprint" "Resistor_THT:R_Axial_DIN0207_L6.3mm_D2.5mm_P2.54mm_Vertical"
 			(at 181.61 67.818 90)
 			(effects
@@
 			)
 		)
-		(property "Footprint" "Resistor_THT:R_Axial_DIN0207_L6.3mm_D2.5mm_P7.62mm_Horizontal"
+		(property "Footprint" "Resistor_THT:R_Axial_DIN0207_L6.3mm_D2.5mm_P2.54mm_Vertical"
 			(at 181.61 65.278 90)
 			(effects

Commit message: update schematics and PCB
Parts:
- U2: value CA56-12CGKWA -> Display_5641BS
Connections:
- net at A1.19 (A0): now also D1.2 (A); no longer SW2.1
- net at A1.20 (A1): now also D2.2 (A); no longer D1.2 (A)
- net at A1.21 (A2): now also D3.2 (A); no longer D2.2 (A)
- net at A1.22 (A3): now also SW2.1; no longer D3.2 (A)
Other:
- moved on the sheet: D1, D2, D3, J10, J11, J12, J13, J4, J5, J6, J7, J8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
