File: PCB Diagrams/Electronics-Power-Consumption-Meter.kicad_sch (KiCad schematic)
At the start: 37 parts, among them J1 Jack_DC, J10 01x02, J11 01x02, J12 01x02, J13 01x02, J2 01x02, J3 01x02, J4 USB_A, J5 Jack_DC, J6 Jack_DC, J7 USB_B_Mini, J8 USB_B_Micro, J9 01x04, SW1 SW_SPDT, SW2 SW_Push, U1 INA219_Module, U2 Display_5641BS

Commit message: update schematics and PCB
Parts:
- removed H4: MountingHole, MountingHole:MountingHole_2mm, symbol Mechanical:MountingHole
Other:
- moved on the sheet: H1, H2, H3
Changed lines of the file:
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@@
 	(symbol
 		(lib_id "Mechanical:MountingHole")
-		(at 209.55 90.17 0)
+		(at 198.12 90.17 0)
 		(unit 1)
 		(exclude_from_sim no)
@@
 		(fields_autoplaced yes)
 		(property "Reference" "H3"
-			(at 212.09 88.8999 0)
+			(at 200.66 88.8999 0)
 			(effects
 				(font
@@
 		)
 		(property "Value" "MountingHole"
-			(at 212.09 91.4399 0)
+			(at 200.66 91.4399 0)
 			(effects
 				(font
@@
 		)
 		(property "Footprint" "MountingHole:MountingHole_2mm"
-			(at 209.55 90.17 0)
-			(effects
-				(font
-					(size 1.27 1.27)
-				)
-				(hide yes)
-			)
-		)
-		(property "Datasheet" "~"
-			(at 209.55 90.17 0)
+			(at 198.12 90.17 0)
+			(effects
+				(font
+					(size 1.27 1.27)
+				)
+				(hide yes)
+			)
+		)
+		(property "Datasheet" "~"
+			(at 198.12 90.17 0)
 			(effects
 				(font
@@
 		)
 		(property "Description" "Mounting Hole without connection"
-			(at 209.55 90.17 0)
+			(at 198.12 90.17 0)
 			(effects
 				(font
@@
 	(symbol
 		(lib_id "Mechanical:MountingHole")
-		(at 209.55 96.52 0)
-		(unit 1)
-		(exclude_from_sim no)
-		(in_bom no)
-		(on_board yes)
-		(dnp no)
-		(fields_autoplaced yes)
-		(property "Reference" "H4"
-			(at 212.09 95.2499 0)
-			(effects
-				(font
-					(size 1.27 1.27)
-				)
-				(justify left)
-			)
-		)
-		(property "Value" "MountingHole"
-			(at 212.09 97.7899 0)
-			(effects
-				(font
-					(size 1.27 1.27)
-				)
-				(justify left)
-			)
-		)
-		(property "Footprint" "MountingHole:MountingHole_2mm"
-			(at 209.55 96.52 0)
-			(effects
-				(font
-					(size 1.27 1.27)
-				)
-				(hide yes)
-			)
-		)
-		(property "Datasheet" "~"
-			(at 209.55 96.52 0)
-			(effects
-				(font
-					(size 1.27 1.27)
-				)
-				(hide yes)
-			)
-		)
-		(property "Description" "Mounting Hole without connection"
-			(at 209.55 96.52 0)
-			(effects
-				(font
-					(size 1.27 1.27)
-				)
-				(hide yes)
-			)
-		)
-		(instances
-			(project "Electronics-Power-Consumption-Meter"
-				(path "/04a21a1e-c762-45c9-8522-5107851ca11f"
-					(reference "H4")
-					(unit 1)
-				)
-			)
-		)
-	)
-	(symbol
-		(lib_id "Mechanical:MountingHole")
-		(at 190.5 96.52 0)
+		(at 217.17 90.17 0)
 		(unit 1)
 		(exclude_from_sim no)
@@
 		(fields_autoplaced yes)
 		(property "Reference" "H2"
-			(at 193.04 95.2499 0)
+			(at 219.71 88.8999 0)
 			(effects
 				(font
@@
 		)
 		(property "Value" "MountingHole"
-			(at 193.04 97.7899 0)
+			(at 219.71 91.4399 0)
 			(effects
 				(font
@@
 		)
 		(property "Footprint" "MountingHole:MountingHole_2mm"
-			(at 190.5 96.52 0)
-			(effects
-				(font
-					(size 1.27 1.27)
-				)
-				(hide yes)
-			)
-		)
-		(property "Datasheet" "~"
-			(at 190.5 96.52 0)
+			(at 217.17 90.17 0)
+			(effects
+				(font
+					(size 1.27 1.27)
+				)
+				(hide yes)
+			)
+		)
+		(property "Datasheet" "~"
+			(at 217.17 90.17 0)
 			(effects
 				(font
@@
 		)
 		(property "Description" "Mounting Hole without connection"
-			(at 190.5 96.52 0)
+			(at 217.17 90.17 0)
 			(effects
 				(font
@@
 	(symbol
 		(lib_id "Mechanical:MountingHole")
-		(at 190.5 90.17 0)
+		(at 179.07 90.17 0)
 		(unit 1)
 		(exclude_from_sim no)
@@
 		(fields_autoplaced yes)
 		(property "Reference" "H1"
-			(at 193.04 88.8999 0)
+			(at 181.61 88.8999 0)
 			(effects
 				(font
@@
 		)
 		(property "Value" "MountingHole"
-			(at 193.04 91.4399 0)
+			(at 181.61 91.4399 0)
 			(effects
 				(font
@@
 		)
 		(property "Footprint" "MountingHole:MountingHole_2mm"
-			(at 190.5 90.17 0)
-			(effects
-				(font
-					(size 1.27 1.27)
-				)
-				(hide yes)
-			)
-		)
-		(property "Datasheet" "~"
-			(at 190.5 90.17 0)
+			(at 179.07 90.17 0)
+			(effects
+				(font
+					(size 1.27 1.27)
+				)
+				(hide yes)
+			)
+		)
+		(property "Datasheet" "~"
+			(at 179.07 90.17 0)
 			(effects
 				(font
@@
 		)
 		(property "Description" "Mounting Hole without connection"
-			(at 190.5 90.17 0)
-			(effects
-				(font
+			(at 179.07 90.17 0)
+			(effects
+				(font
